File: ridge-3/esc/ridge3-esc.kicad_pcb (KiCad board)
At the start: 8 copper layers, 36 x 36 mm, 193 parts, among them Q1AH ISZ023N06LM6, Q1AL ISZ023N06LM6, Q1BH ISZ023N06LM6, Q1BL ISZ023N06LM6, Q1CH ISZ023N06LM6, Q1CL ISZ023N06LM6, Q2AH ISZ023N06LM6, Q2AL ISZ023N06LM6, Q2BH ISZ023N06LM6, Q2BL ISZ023N06LM6, Q2CH ISZ023N06LM6, Q2CL ISZ023N06LM6, Q3AH ISZ023N06LM6, Q3AL ISZ023N06LM6, Q3BH ISZ023N06LM6, Q3BL ISZ023N06LM6, Q3CH ISZ023N06LM6, Q3CL ISZ023N06LM6, Q4AH ISZ023N06LM6, Q4AL ISZ023N06LM6, Q4BH ISZ023N06LM6, Q4BL ISZ023N06LM6, Q4CH ISZ023N06LM6, Q4CL ISZ023N06LM6

Commit message: ESC rebuilt with the 3.3 V hub capacitor on the bottom: DRC 0, every gate passed
make.py --reroute: the template channel and the four whole-board tries
routed; try 0 kept (0 nets open).  Its clean-up left one DRV_EN overshoot
the old trim could not take (fixed in cleanup.py), so the run's last
steps were redone with make.py --finish on the same routing: clean-up
0 / 0 / 0, artwork, final DRC 0 errors, 0 warnings, 0 unconnected; nets
match circuit.py pad for pad; BOM and CPL list exactly the 159 assembled
parts.  The stack lead's 3.3 V pad now has its '3V3' label; the SWD clock
pads read 'C'; the firmware name stays off (no room), as before.

Co-Authored-By: Claude Opus 5.5 <noreply@anthropic.com>
Claude-Session: https://claude.ai/code/session_01MaVFAzoExts7u2gmCraXFC
Parts:
- C5: moved to B.Cu
- moved C5 2.87 mm to (102.5, 97.6)
Routing:
- net ESC_3V3: track 85.9 -> 158.8 mm, vias 9 -> 10
- net M4_CMP_A: track 53.4 -> 81.5 mm, vias 5 -> 6
- net M3_CMP_A: track 73.9 -> 83.9 mm
- net M4_HB: track 12.7 -> 4.68 mm
- net M3_LA: track 3.24 -> 8.39 mm
- net M3_LB: track 9.58 -> 5.13 mm
- net CUR: track 92.4 -> 95.9 mm
- net M4_LA: track 6.59 -> 3.24 mm
- net M4_A: track 13.0 -> 9.69 mm
- net M1_A: track 13.0 -> 9.69 mm
- net DRV_EN: track 36.7 -> 33.6 mm, vias 4 -> 2
- net M4_SIG: track 13.5 -> 16.0 mm, vias 3 -> 2
- net M2_CMP_A: track 32.6 -> 35.0 mm, vias 3 -> 4
- net M4_GHB: track 9.77 -> 11.9 mm
- net M2_GHB: track 9.77 -> 11.9 mm
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
Commit message: ESC outputs and 3 x 2 panel with the 18k IDRIVE resistors: every gate passed
make.py esc (no new layout): the four IDRIVE resistors' value and LCSC
fields from circuit.py, DRC 0 / 0 / 0, nets pad for pad, BOM and CPL of
the 159 assembled parts, and the production panel rebuilt on this board
(it was last built before the 3.3 V rework): DRC 6 x the board's own,
every copy's Gerbers, BOM and CPL equal to the board's.

Co-Authored-By: Claude Opus 5.5 <noreply@anthropic.com>
Claude-Session: https://claude.ai/code/session_01MaVFAzoExts7u2gmCraXFC
Parts:
- R21, R33, R45, R9: value 75k -> 18k
Changed lines of the file:
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@@
 			)
 		)
-		(property "Value" "75k"
+		(property "Value" "18k"
 			(at 0 1.05 0)
 			(layer "F.Fab")
@@
 			)
 		)
-		(property "LCSC" "C295816"
+		(property "LCSC" "C295780"
 			(at 0 0 0)
 			(layer "F.Fab")
@@
 			)
 		)
-		(property "Value" "75k"
+		(property "Value" "18k"
 			(at 0 1.05 270)
 			(layer "F.Fab")
@@
 			)
 		)
-		(property "LCSC" "C295816"
+		(property "LCSC" "C295780"
 			(at 0 0 270)
 			(layer "F.Fab")
@@
 			)
 		)
-		(property "Value" "75k"
+		(property "Value" "18k"
 			(at 0 1.05 180)
 			(layer "F.Fab")
@@
 			)
 		)
-		(property "LCSC" "C295816"
+		(property "LCSC" "C295780"
 			(at 0 0 180)
 			(layer "F.Fab")
@@
 			)
 		)
-		(property "Value" "75k"
+		(property "Value" "18k"
 			(at 0 1.05 90)
 			(layer "F.Fab")
@@
 			)
 		)
-		(property "LCSC" "C295816"
+		(property "LCSC" "C295780"
 			(at 0 0 90)
 			(layer "F.Fab")

Commit message: ESC: IDRIVE back to 60/120 mA (75 kOhm), the owner's choice of heat
30/60 mA kept the high side's turn-off undershoot at SHx to -6.2 V, inside
the DRV8320H's -7 V, but doubled the switching energy and nearly doubled
the dead time: on a 50 C day the throttle AM32's temperature limit lets the
stack hold fell from 34 to 28 %.  60/120 mA takes the heat back and accepts
-9.5 V at 30 A in the 5 nH loop (-7.8 V at 20 A) for 200 ns; STRESS.md
keeps judging it against the driver's -7 V.  The four IDRIVE resistors
(R9, R21, R33, R45) take their value and LCSC number from circuit.py;
the copper is unchanged.

Co-Authored-By: Claude Opus 5.5 <noreply@anthropic.com>
Claude-Session: https://claude.ai/code/session_01MaVFAzoExts7u2gmCraXFC
Parts:
- R21, R33, R45, R9: value 18k -> 75k
Changed lines of the file:
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@@
 			)
 		)
-		(property "Value" "18k"
+		(property "Value" "75k"
 			(at 0 1.05 0)
 			(layer "F.Fab")
@@
 			)
 		)
-		(property "LCSC" "C295780"
+		(property "LCSC" "C295816"
 			(at 0 0 0)
 			(layer "F.Fab")
@@
 			)
 		)
-		(property "Value" "18k"
+		(property "Value" "75k"
 			(at 0 1.05 270)
 			(layer "F.Fab")
@@
 			)
 		)
-		(property "LCSC" "C295780"
+		(property "LCSC" "C295816"
 			(at 0 0 270)
 			(layer "F.Fab")
@@
 			)
 		)
-		(property "Value" "18k"
+		(property "Value" "75k"
 			(at 0 1.05 180)
 			(layer "F.Fab")
@@
 			)
 		)
-		(property "LCSC" "C295780"
+		(property "LCSC" "C295816"
 			(at 0 0 180)
 			(layer "F.Fab")
@@
 			)
 		)
-		(property "Value" "18k"
+		(property "Value" "75k"
 			(at 0 1.05 90)
 			(layer "F.Fab")
@@
 			)
 		)
-		(property "LCSC" "C295780"
+		(property "LCSC" "C295816"
 			(at 0 0 90)
 			(layer "F.Fab")
