File: print-hub/v1/print-hub.kicad_pcb (KiCad board)
At the start: 4 copper layers, 104 x 66 mm, 135 parts, among them J1 USB-C, J101 USB-A, J2 USB-C, J201 USB-A, J301 USB-A, J401 USB-A, J501 USB-A, SW1 button, SW2 button, U1 HUSB238, U101 TPS25200, U102 INA180A2, U2 SY8368A, U201 TPS25200, U202 INA180A2, U3 USBLC6-2SC6, U301 TPS25200, U302 INA180A2, U4 AP2112K-3.3, U401 TPS25200, U402 INA180A2, U5 ESP32-S3-WROOM-1-N8, U501 TPS25200, U502 INA180A2

Commit message: print-hub v1: final routed board and fab files
DRC 0 / 0 / 0, nets equal circuit.py, 128 assembled parts in 34 BOM
lines. Renders and STEP with the connector models on their lands.

Co-Authored-By: Claude Opus 5.5 <noreply@anthropic.com>
Claude-Session: https://claude.ai/code/session_01AiCo3BFL3vgJ9qSJmY4RFn
Parts:
- removed the C101 at (60.7, 112.3)
- removed the C201 at (78.7, 112.3)
- removed the C301 at (96.7, 112.3)
- removed the C401 at (114.7, 112.3)
- removed the C501 at (132.7, 112.3)
- removed the R105 at (69.4, 113.4)
- removed the R17 at (121.0, 80.4)
- removed the R205 at (87.4, 113.4)
- removed the R305 at (105.4, 113.4)
- removed the R405 at (123.4, 113.4)
- removed the R505 at (141.4, 113.4)
- added C102: 22uF, C_1206_3216Metric, F.Cu at (59.0, 112.8)
- added C105: 22uF, C_1206_3216Metric, F.Cu at (60.4, 118.0)
- added C18: 100nF, C_0402_1005Metric, F.Cu at (121.0, 77.8)
- added C20: 100nF, C_0402_1005Metric, F.Cu at (148.6, 90.0)
- added C202: 22uF, C_1206_3216Metric, F.Cu at (77.0, 112.8)
- added C205: 22uF, C_1206_3216Metric, F.Cu at (78.4, 118.0)
- added C302: 22uF, C_1206_3216Metric, F.Cu at (95.0, 112.8)
- added C305: 22uF, C_1206_3216Metric, F.Cu at (96.4, 118.0)
- added C402: 22uF, C_1206_3216Metric, F.Cu at (113.0, 112.8)
- added C405: 22uF, C_1206_3216Metric, F.Cu at (114.4, 118.0)
- added C502: 22uF, C_1206_3216Metric, F.Cu at (131.0, 112.8)
- added C505: 22uF, C_1206_3216Metric, F.Cu at (132.4, 118.0)
- C101: renamed from C102; value 22uF -> 100nF; footprint C_1206_3216Metric -> C_0402_1005Metric
- C104: renamed from C105; value 22uF -> 100nF; footprint C_1206_3216Metric -> C_0402_1005Metric
- C16: value 22uF -> 10uF
- C17: value 100nF -> 22uF; footprint C_0402_1005Metric -> C_0603_1608Metric
- C19: value 100nF -> 1uF
- C201: renamed from C202; value 22uF -> 100nF; footprint C_1206_3216Metric -> C_0402_1005Metric
- C204: renamed from C205; value 22uF -> 100nF; footprint C_1206_3216Metric -> C_0402_1005Metric
- C301: renamed from C302; value 22uF -> 100nF; footprint C_1206_3216Metric -> C_0402_1005Metric
- C304: renamed from C305; value 22uF -> 100nF; footprint C_1206_3216Metric -> C_0402_1005Metric
- C401: renamed from C402; value 22uF -> 100nF; footprint C_1206_3216Metric -> C_0402_1005Metric
- C404: renamed from C405; value 22uF -> 100nF; footprint C_1206_3216Metric -> C_0402_1005Metric
- C501: renamed from C502; value 22uF -> 100nF; footprint C_1206_3216Metric -> C_0402_1005Metric
- C504: renamed from C505; value 22uF -> 100nF; footprint C_1206_3216Metric -> C_0402_1005Metric
- R105: renamed from C104; value 100nF -> 1k; footprint C_0402_1005Metric -> R_0402_1005Metric
- R17: renamed from C18; value 1uF -> 10k; footprint C_0402_1005Metric -> R_0402_1005Metric
- R205: renamed from C204; value 100nF -> 1k; footprint C_0402_1005Metric -> R_0402_1005Metric
- R305: renamed from C304; value 100nF -> 1k; footprint C_0402_1005Metric -> R_0402_1005Metric
- R405: renamed from C404; value 100nF -> 1k; footprint C_0402_1005Metric -> R_0402_1005Metric
- R505: renamed from C504; value 100nF -> 1k; footprint C_0402_1005Metric -> R_0402_1005Metric
- moved C19 30.4 mm to (119.8, 80.4)
- moved C16 26.6 mm to (96.0, 84.4)
- moved C104 11.2 mm to (70.6, 113.4), turned to 90 degrees
- moved C204 11.2 mm to (88.6, 113.4), turned to 90 degrees
- moved C304 11.2 mm to (106.6, 113.4), turned to 90 degrees
- moved C404 11.2 mm to (124.6, 113.4), turned to 90 degrees
- moved C504 11.2 mm to (142.6, 113.4), turned to 90 degrees
- moved C15 7.61 mm to (88.4, 84.0)
- moved C14 5.34 mm to (87.2, 78.8)
- moved C17 2.60 mm to (121.0, 75.2)
- moved C101 1.77 mm to (60.7, 112.3)
- moved C201 1.77 mm to (78.7, 112.3)
- moved C301 1.77 mm to (96.7, 112.3)
- moved C401 1.77 mm to (114.7, 112.3)
- moved C501 1.77 mm to (132.7, 112.3)
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Connections:
- C104 pad 1: VBUS1 -> IS1
- C14 pad 1: VLOGIC -> VBUS_DATA
- C15 pad 1: +3V3 -> VLOGIC
- C19 pad 1: VLOGIC -> ESP_EN
- C204 pad 1: VBUS2 -> IS2
- C304 pad 1: VBUS3 -> IS3
- C404 pad 1: VBUS4 -> IS4
- C504 pad 1: VBUS5 -> IS5
- R105 pad 1: IS1 -> ISA1
- R105 pad 2: GND -> IS1
- R17 pad 2: GND -> +3V3
- R205 pad 1: IS2 -> ISA2
- R205 pad 2: GND -> IS2
- R305 pad 1: IS3 -> ISA3
- R305 pad 2: GND -> IS3
- R405 pad 1: IS4 -> ISA4
- R405 pad 2: GND -> IS4
- R505 pad 1: IS5 -> ISA5
- R505 pad 2: GND -> IS5
Routing:
- net SDA: track 83.9 -> 94.8 mm, vias 4 -> 2
- net +3V3: track 249.2 -> 239.0 mm
- net VLOGIC: track 200.2 -> 210.3 mm, vias 6 -> 3
- net USB_DN: track 50.2 -> 60.1 mm
- net USB_DP: track 50.5 -> 60.3 mm
- net RXD0: track 34.3 -> 26.7 mm
- net ISA3: track 9.93 -> 2.58 mm, vias 2 -> 0
- net IS1: track 100.8 -> 94.4 mm
- net CC2_DATA: track 4.68 -> 9.85 mm
- net BUCK_LX: track 7.55 -> 2.55 mm
- net BOOT: track 36.9 -> 32.7 mm, vias 2 -> 0
- net FLT3: track 40.9 -> 37.3 mm
- net BUCK_FB: track 17.5 -> 14.3 mm
- net FLT5: track 39.3 -> 36.2 mm, vias 0 -> 2
- net VBUS_IN: track 32.6 -> 35.7 mm, vias 2 -> 6
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- added copper zone on F.Cu, net BUCK_LX
