File: mesh-radio/v1/schematic/system.kicad_sch (KiCad schematic)
At the start: 15 parts, among them SW1 JS102011SAQN, U6 TPS22965DSGR, U7 TPS62840YBGR

Commit message: Mesh Radio v1: fix every design-review finding, add the part audit
An independent review of the schematic found two critical and nine further
issues; all are fixed in src/circuit.py:
- reverse-battery FET gate now returns to the cell's own minus terminal, so
  a backwards cell stays isolated even while USB/solar/drone power the board
- solar and drone inputs: reverse-blocking Schottky + 22 V flat-clamp TVS
  (the 15 V TVS would have failed on a 12 V panel); 4.7 V clamp on every
  eFuse EN/UVLO pin so 20 V on an input stays inside its rating
- ideal diode (LM66100) holds VSYS on the cell when a 3 W burst trips the
  charger's 3.0 V battery disconnect
- charge LED moved to STAT2 (charging), USB cut-off lowered to 5.4 V,
  charger /CE on a GPIO for firmware temperature control, -40 C TCXO,
  power mux on only with the amplifier, header VSYS pin removed
- firmware ceilings documented: SX1262 +20 dBm, amplifier 3.6 V by default

docs/part-audit.md: all 125 lines checked at DigiKey and LCSC (genuine
LCSC numbers, DigiKey numbers, second sources for out-of-stock lines);
parts cost about $76 at 10 boards, $58 at 100.

Schematic regenerated: ERC 0 violations, netlist equals circuit.py.

Co-Authored-By: Claude Opus 5.5 <noreply@anthropic.com>
Claude-Session: https://claude.ai/code/session_015TBB2ThqxHSgA8MkFosmn9
Parts:
- removed U6: TPS22965DSGR, og:UDFN-8_L2.0-W2.0-P0.50-TL-EP, symbol og:TPS22965
- added U8: TPS62840YBGR, og:DSBGA-6_L1.4-W1.0-R2-C3-P0.40-BL, symbol og:TPS62840
- C16: DigiKey (none) -> 490-3244-1-ND
- C17: DigiKey (none) -> 1276-1184-1-ND
- C18, C20, C21: DigiKey (none) -> 1276-1192-1-ND
- C19: DigiKey (none) -> 1276-1044-1-ND
- L1: DigiKey (none) -> 490-17728-1-ND
- R33: DigiKey (none) -> 311-1.00MLRCT-ND
- R34: DigiKey (none) -> YAG3079CT-ND
- SW1: DigiKey (none) -> 401-1999-1-ND
- U7: value TPS62840YBGR -> TPS22965DSGR; footprint og:DSBGA-6_L1.4-W1.0-R2-C3-P0.40-BL -> og:UDFN-8_L2.0-W2.0-P0.50-TL-EP; symbol og:TPS62840 -> og:TPS22965; DigiKey (none) -> 296-39362-1-ND; LCSC C2071139 -> C122837; MPN TPS62840YBGR -> TPS22965DSGR
Connections:
- net 3V3: now also U8.A2 (VOS); no longer U7.A2 (VOS)
- net BUCK_SW: now also U8.B2 (SW); no longer U7.B2 (SW)
- net BUCK_VSET: now also U8.C2 (VSET); no longer U7.C2 (VSET)
- net GND: now also U7.5 (GND), U7.9 (GND (EP)), U8.A1 (GND); no longer U7.A1 (GND)
- net PWR_ON: now also U7.3 (ON)
- net SW_CT: now also U7.6 (CT)
- net VSYS: now also U7.1 (VIN), U7.2 (VIN), U7.4 (VBIAS)
- net VSYS_SW: now also U7.7 (VOUT), U7.8 (VOUT), U8.B1 (VIN), U8.C1 (EN); no longer U7.B1 (VIN), U7.C1 (EN)
Changed lines of the file:
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@@
+			)
+		)
+		(property "DigiKey" "401-1999-1-ND"
+			(at 43.18 48.26 0)
+			(effects
+				(font
+					(size 1.27 1.27)
+				)
+				(hide yes)
 			)
 		)
@@
 		(on_board yes)
 		(dnp no)
-		(property "Reference" "U6"
+		(property "Reference" "U7"
 			(at 76.2 41.68 0)
 			(effects
@@
 			)
 		)
+		(property "DigiKey" "296-39362-1-ND"
+			(at 86.36 50.8 0)
+			(effects
+				(font
+					(size 1.27 1.27)
+				)
+				(hide yes)
+			)
+		)
 		(property "LCSC" "C122837"
 			(at 86.36 50.8 0)
@@
 			(project "mesh-radio"
 				(path "/1e0df660-60b5-6ed0-6a2a-f5098e72ebfd/2f3f0b85-467d-aba7-63bd-0d0b1c38f73c"
-					(reference "U6")
+					(reference "U7")
 					(unit 1)
 				)
@@
 		(on_board yes)
 		(dnp no)
-		(property "Reference" "U7"
+		(property "Reference" "U8"
 			(at 128.27 41.68 0)
 			(effects
@@
 			)
 		)
+		(property "DigiKey" "296-TPS62840YBGRCT-ND"
+			(at 134.62 48.26 0)
+			(effects
+				(font
+					(size 1.27 1.27)
+				)
+				(hide yes)
+			)
+		)
 		(property "LCSC" "C2071139"
 			(at 134.62 48.26 0)
@@
 			(project "mesh-radio"
 				(path "/1e0df660-60b5-6ed0-6a2a-f5098e72ebfd/2f3f0b85-467d-aba7-63bd-0d0b1c38f73c"
-					(reference "U7")
+					(reference "U8")
 					(unit 1)
 				)
@@
 			)
 		)
+		(property "DigiKey" "311-1.00MLRCT-ND"
+			(at 25.4 96.52 0)
+			(effects
+				(font
+					(size 1.27 1.27)
+				)
+				(hide yes)
+			)
+		)
 		(property "LCSC" "C138033"
 			(at 25.4 96.52 0)
@@
 			)
 		)
+		(property "DigiKey" "490-3244-1-ND"
+			(at 38.1 96.52 0)
+			(effects
+				(font
+					(size 1.27 1.27)
+				)
+				(hide yes)
+			)
+		)
 		(property "LCSC" "C76947"
 			(at 38.1 96.52 0)
@@
 			)
 		)
+		(property "DigiKey" "1276-1184-1-ND"
+			(at 50.8 91.44 0)
+			(effects
+				(font
+					(size 1.27 1.27)
+				)
+				(hide yes)
+			)
+		)
 		(property "LCSC" "C29936"
 			(at 50.8 91.44 0)
@@
 			)
 		)
+		(property "DigiKey" "1276-1192-1-ND"
+			(at 63.5 91.44 0)
+			(effects
+				(font
+					(size 1.27 1.27)
+				)
+				(hide yes)
+			)
+		)
 		(property "LCSC" "C19702"
 			(at 63.5 91.44 0)
@@
 		)
 		(property "Manufacturer" "Yageo"
+			(at 76.2 99.06 0)
+			(effects
+				(font
+					(size 1.27 1.27)
+				)
+				(hide yes)
+			)
+		)
+		(property "DigiKey" "YAG3079CT-ND"
 			(at 76.2 99.06 0)
 			(effects
@@
 			)
 		)
+		(property "DigiKey" "1276-1044-1-ND"
+			(at 88.9 91.44 0)
+			(effects
+				(font
+					(size 1.27 1.27)
+				)
+				(hide yes)
+			)
+		)
 		(property "LCSC" "C1705"
 			(at 88.9 91.44 0)
@@
 		)
 		(property "Manufacturer" "Murata"
+			(at 101.6 91.44 0)
+			(effects
+				(font
+					(size 1.27 1.27)
+				)
+				(hide yes)
+			)
+		)
+		(property "DigiKey" "490-17728-1-ND"
 			(at 101.6 91.44 0)
 			(effects
@@
 			)
 		)
+		(property "DigiKey" "1276-1192-1-ND"
+			(at 114.3 91.44 0)
+			(effects
+				(font
+					(size 1.27 1.27)
+				)
+				(hide yes)
+			)
+		)
 		(property "LCSC" "C19702"
 			(at 114.3 91.44 0)
@@
 			(at 127 91.44 0)
 			(effects
+				(font
+					(size 1.27 1.27)
+				)
+				(hide yes)
+			)
+		)
+		(property "DigiKey" "1276-1192-1-ND"
+			(at 127 91.44 0)
+			(effects

Commit message: Mesh radio v1: power-path and firmware rework in progress (snapshot)
Co-Authored-By: Claude Opus 5.5 <noreply@anthropic.com>
Claude-Session: https://claude.ai/code/session_015TBB2ThqxHSgA8MkFosmn9
Parts:
- removed C20, C21: 10uF, og:C_0603, symbol Device:C
- removed R33: 1M, og:R_0402, symbol Device:R
- removed R34: 267k, og:R_0402, symbol Device:R
- removed U8: TPS62840YBGR, og:DSBGA-6_L1.4-W1.0-R2-C3-P0.40-BL, symbol og:TPS62840
- added C15: 1uF, og:C_0603, symbol Device:C
- added R38: 1M, og:R_0402, symbol Device:R
- added R39: 267k, og:R_0402, symbol Device:R
- C16: value 1nF -> 10uF; footprint og:C_0402 -> og:C_0603; DigiKey 490-3244-1-ND -> 1276-1192-1-ND; LCSC C76947 -> C19702; MPN GRM1555C1H102JA01D -> CL10A106KP8NNNC; Manufacturer Murata -> Samsung Electro-Mechanics
- C17: value 1uF -> 4.7uF; DigiKey 1276-1184-1-ND -> 1276-1044-1-ND; LCSC C29936 -> C1705; MPN CL10B105KA8NNNC -> CL10A475KP8NNNC
- C19: value 4.7uF -> 10uF; DigiKey 1276-1044-1-ND -> 1276-1192-1-ND; LCSC C1705 -> C19702; MPN CL10A475KP8NNNC -> CL10A106KP8NNNC
- U7: value TPS22965DSGR -> TPS62840YBGR; footprint og:UDFN-8_L2.0-W2.0-P0.50-TL-EP -> og:DSBGA-6_L1.4-W1.0-R2-C3-P0.40-BL; symbol og:TPS22965 -> og:TPS62840; DigiKey 296-39362-1-ND -> 296-TPS62840YBGRCT-ND; LCSC C122837 -> C2071139; MPN TPS22965DSGR -> TPS62840YBGR
Connections:
- net 3V3: now also C18.1, C19.1, U7.A2 (VOS)
- net BUCK_SW: now also U7.B2 (SW)
- net BUCK_VSET: now also U7.C2 (VSET), R39.1
- net GND: now also U7.A1 (GND), C15.2, R38.2, R39.2; no longer U7.5 (GND), U7.9 (GND (EP))
- net PWR_ON: now also U7.C1 (EN), R38.1; no longer U7.3 (ON)
- net VSYS: now also C16.1, U7.B1 (VIN), C15.1; no longer U7.1 (VIN), U7.2 (VIN), U7.4 (VBIAS)
- removed net SW_CT: C16.1, U7.6 (CT)
- removed net VSYS_SW: C18.1, C19.1, U7.7 (VOUT), U7.8 (VOUT)
Other:
- note added: "The slide switch drives only enables (3.3 V buck, cell bypass); charging works with the board off."
- note removed: "The slide switch only drives the load switch enable; charging works with the board switched off."
- moved on the sheet: C16, C17, C18, C19, L1, TP1, TP2, TP3
