File: mesh-radio/v1/schematic/pa_power.kicad_sch (KiCad schematic)
At the start: 28 parts, among them Q3 SSM3K56ACT, U14 TPS2121RUXR, U15 TPS63810YFFR, U16 TLV75528PDQNR, U17 TMP1075NDRLR

Commit message: Mesh radio v1: power-path and firmware rework in progress (snapshot)
Co-Authored-By: Claude Opus 5.5 <noreply@anthropic.com>
Claude-Session: https://claude.ai/code/session_015TBB2ThqxHSgA8MkFosmn9
Parts:
- removed C98: 1uF, og:C_0402, symbol Device:C
- removed C99: 100nF, og:C_0402, symbol Device:C
- removed Q3: SSM3K56ACT, og:SOT-883, symbol og_device:Q_NMOS_NMOS
- removed R48: 562k, og:R_0402, symbol Device:R
- removed R49: 301k, og:R_0402, symbol Device:R
- removed R50, R52: 1M, og:R_0402, symbol Device:R
- removed R51: 22.1k, og:R_0402, symbol Device:R
- removed U17: TMP1075NDRLR, og:SOT-563_L1.6-W1.2-P0.50-LS1.6-BR, symbol og:TMP1075
- added C86: 10nF, og:C_0402, symbol Device:C
- added C87: 1uF, og:C_0603, symbol Device:C
- added Q4, Q5: SSM3K56ACT, og:SOT-883, symbol og_device:Q_NMOS_NMOS
- added R58: 1M, og:R_0402, symbol Device:R
- added R59, R60: 100k, og:R_0402, symbol Device:R
- added R61, R62: 4.7k, og:R_0402, symbol Device:R
- added U13: TPS2121RUXR, og:VQFN-12_TPS2121RUX, symbol og:TPS2121
- C88: value 10nF -> 1uF; footprint og:C_0402 -> og:C_0603; DigiKey 1276-1028-1-ND -> 1276-1184-1-ND; LCSC C15195 -> C29936; MPN CL05B103KB5NNNC -> CL10B105KA8NNNC
- C89, C90: value 1uF -> 22uF; footprint og:C_0603 -> og:C_0805; DigiKey 1276-1184-1-ND -> (none); LCSC C29936 -> C86817; MPN CL10B105KA8NNNC -> GRM21BR61C226ME44L; Manufacturer Samsung Electro-Mechanics -> Murata
- C91: value 22uF -> 10uF; DigiKey (none) -> 1276-2891-1-ND; LCSC C86817 -> C15850; MPN GRM21BR61C226ME44L -> CL21A106KAYNNNE; Manufacturer Murata -> Samsung Electro-Mechanics
- C92: value 22uF -> 47uF; footprint og:C_0805 -> og:C_1206; DigiKey (none) -> 445-8037-1-ND; LCSC C86817 -> C2167997; MPN GRM21BR61C226ME44L -> C3216X7S0J476M160AC; Manufacturer Murata -> TDK
- C93: value 10uF -> 47uF; footprint og:C_0805 -> og:C_1206; DigiKey 1276-2891-1-ND -> 445-8037-1-ND; LCSC C15850 -> C2167997; MPN CL21A106KAYNNNE -> C3216X7S0J476M160AC; Manufacturer Samsung Electro-Mechanics -> TDK
- C94: value 47uF -> 100nF; footprint og:C_0805 -> og:C_0402; DigiKey 1276-1852-1-ND -> 1276-1001-1-ND; LCSC C16780 -> C1525; MPN CL21A476MQYNNNE -> CL05B104KO5NNNC
- C95: value 47uF -> 1uF; footprint og:C_0805 -> og:C_0402; DigiKey 1276-1852-1-ND -> 1276-1067-1-ND; LCSC C16780 -> C29266; MPN CL21A476MQYNNNE -> CL05A105KO5NNNC
- C96: value 100nF -> 1uF; DigiKey 1276-1001-1-ND -> 1276-1067-1-ND; LCSC C1525 -> C29266; MPN CL05B104KO5NNNC -> CL05A105KO5NNNC
- C97: value 1uF -> 100nF; DigiKey 1276-1067-1-ND -> 1276-1001-1-ND; LCSC C29266 -> C1525; MPN CL05A105KO5NNNC -> CL05B104KO5NNNC
- R53: value 1M -> 562k; DigiKey 311-1.00MLRCT-ND -> 311-562KLRCT-ND; LCSC C138033 -> C273337; MPN RC0402FR-071ML -> RC0402FR-07562KL
- R54: value 100k -> 374k; DigiKey 311-100KLRCT-ND -> YAG3136CT-ND; LCSC C60491 -> C185423; MPN RC0402FR-07100KL -> RC0402FR-07374KL
- R55: value 100k -> 1M; DigiKey 311-100KLRCT-ND -> 311-1.00MLRCT-ND; LCSC C60491 -> C138033; MPN RC0402FR-07100KL -> RC0402FR-071ML
- R56: value 4.7k -> 1M; DigiKey 311-4.7KLRCT-ND -> 311-1.00MLRCT-ND; LCSC C105871 -> C138033; MPN RC0402FR-074K7L -> RC0402FR-071ML
- R57: value 4.7k -> 22.1k; DigiKey 311-4.7KLRCT-ND -> 311-22.1KLRCT-ND; LCSC C105871 -> C163478; MPN RC0402FR-074K7L -> RC0402FR-0722K1L
- U14: value TPS2121RUXR -> TPS63810YFFR; footprint og:VQFN-12_TPS2121RUX -> og:DSBGA-15_L2.2-W1.4-R3-V5-P0.40-BL; symbol og:TPS2121 -> og:TPS63810; DigiKey 296-53410-1-ND -> 296-TPS63810YFFRCT-ND; LCSC C485916 -> C1852139; MPN TPS2121RUXR -> TPS63810YFFR
- U15: value TPS63810YFFR -> TLV75528PDQNR; footprint og:DSBGA-15_L2.2-W1.4-R3-V5-P0.40-BL -> og:X2SON-4_L1.0-W1.0-P0.65-TL-EP; symbol og:TPS63810 -> og:TLV75528; DigiKey 296-TPS63810YFFRCT-ND -> 296-TLV75528PDQNRCT-ND; LCSC C1852139 -> C2865384; MPN TPS63810YFFR -> TLV75528PDQNR
- U16: value TLV75528PDQNR -> TMP1075NDRLR; footprint og:X2SON-4_L1.0-W1.0-P0.65-TL-EP -> og:SOT-563_L1.6-W1.2-P0.50-LS1.6-BR; symbol og:TLV75528 -> og:TMP1075; DigiKey 296-TLV75528PDQNRCT-ND -> 296-TMP1075NDRLRCT-ND; LCSC C2865384 -> C3663690; MPN TLV75528PDQNR -> TMP1075NDRLR
Connections:
- net 3V3: now also C95.1, U15.4 (IN), U16.5 (V+), R60.2, R61.2, R62.2; no longer R55.2, R56.2, R57.2, U16.4 (IN)
- net BAT_P: now also R53.1, R56.1, C87.1, U13.7 (IN1); no longer C89.1, U14.7 (IN1)
- net GND: now also R55.2, R57.2, U14.B1 (VSEL), U14.C1 (AGND), U14.C2 (GND), U14.C3 (GND), U15.2 (GND), U15.5 (GND (EP)), U16.4 (A0), C86.2, C87.2, Q4.2 (S), Q5.2 (S), R58.2, R59.2, U13.12 (GND), U13.3 (CP2), U13.9 (ST); no longer R53.2, U14.12 (GND), U14.3 (CP2), U14.9 (ST), U15.C1 (AGND), U15.C2 (GND), U15.C3 (GND), U16.5 (GND (EP))
- net I2C_SCL: now also U14.D1 (SCL), U16.1 (SCL), R62.1; no longer R57.1, U15.D1 (SCL)
- net I2C_SDA: now also U14.E1 (SDA), U16.6 (SDA), R61.1; no longer R56.1, U15.E1 (SDA)
- net MUX_ILM: now also R57.1, U13.10 (ILM); no longer U14.10 (ILM)
- net MUX_OFF: now also R56.2, Q5.3 (D), U13.4 (OV2), U13.5 (OV1); no longer U14.4 (OV2), U14.5 (OV1)
- net MUX_PR1: now also R53.2, R54.1, Q4.3 (D), U13.6 (PR1); no longer U14.6 (PR1)
- net MUX_SS: now also C86.1, U13.11 (SS); no longer C88.1, U14.11 (SS)
- net PA_APC: now also C96.1, U15.1 (OUT); no longer U16.1 (OUT)
- net PA_EN: now also U15.3 (EN), R59.1; no longer R54.1, U16.3 (EN)
- net PA_IN: now also C89.1, C90.1, U14.A2 (VIN), U14.A3 (VIN), U13.1 (OUT), U13.8 (OUT); no longer C92.1, C93.1, U14.1 (OUT), U14.8 (OUT), U15.A2 (VIN), U15.A3 (VIN)
- net PA_LX1: now also U14.B2 (LX1), U14.B3 (LX1); no longer U15.B2 (LX1), U15.B3 (LX1)
- net PA_LX2: now also U14.D2 (LX2), U14.D3 (LX2); no longer U15.D2 (LX2), U15.D3 (LX2)
- net PA_PWR_EN: now also U14.A1 (EN), Q5.1 (G), R58.1; no longer U15.A1 (EN)
- net TEMP_ALERT: now also U16.3 (ALERT), R60.1; no longer R55.1
- net VPA: now also C92.1, C93.1, U14.E2 (VOUT), U14.E3 (VOUT); no longer C95.1, C96.1, U15.E2 (VOUT), U15.E3 (VOUT)
- net VSYS: now also C88.1, U13.2 (IN2); no longer C90.1, U14.2 (IN2)
- removed net PA_VSEL: R53.1, U15.B1 (VSEL)
- new net PA_SRC_SYS: Q4.1 (G), R55.1
Other:
- note added: "Amplifier runs from the battery through a power mux (battery first down to 2.6 V; firmware selects charger SYS when no cell is fitted), then a TPS63810 buck-boost (I2C 0x75): 2.7 V for 1 W, 4.0 V for 3 W."
- note removed: "Amplifier runs from the battery through a power mux (charger SYS only when no battery), then a TPS63810 buck-boost set over I2C (0x75): ~2.7 V for 1 W, up to 4.0 V for 3 W."
- moved on the sheet: C88, C89, C90, C91, C92, C93, C94, C95, C96, C97, R53, R54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

Commit message: Mesh Radio v1 schematic: regenerated (gate clamp, NTC part); ERC 0, netlist equal
Co-Authored-By: Claude Opus 5.5 <noreply@anthropic.com>
Claude-Session: https://claude.ai/code/session_015TBB2ThqxHSgA8MkFosmn9
Parts:
- C89, C90: DigiKey (none) -> 490-10747-1-ND
Changed lines of the file:
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@@
+			)
+		)
+		(property "DigiKey" "490-10747-1-ND"
+			(at 127 104.14 0)
+			(effects
+				(font
+					(size 1.27 1.27)
+				)
+				(hide yes)
 			)
 		)
@@
 			(at 139.7 104.14 0)
 			(effects
+				(font
+					(size 1.27 1.27)
+				)
+				(hide yes)
+			)
+		)
+		(property "DigiKey" "490-10747-1-ND"
+			(at 139.7 104.14 0)
+			(effects
