File: mesh-radio/v1/schematic/radio.kicad_sch (KiCad schematic)
At the start: 25 parts, among them U9 SX1262IMLTRT, Y3 ECS-TXO-20CSMV4-320-AY-TR

Commit message: Mesh Radio v1: fix every design-review finding, add the part audit
An independent review of the schematic found two critical and nine further
issues; all are fixed in src/circuit.py:
- reverse-battery FET gate now returns to the cell's own minus terminal, so
  a backwards cell stays isolated even while USB/solar/drone power the board
- solar and drone inputs: reverse-blocking Schottky + 22 V flat-clamp TVS
  (the 15 V TVS would have failed on a 12 V panel); 4.7 V clamp on every
  eFuse EN/UVLO pin so 20 V on an input stays inside its rating
- ideal diode (LM66100) holds VSYS on the cell when a 3 W burst trips the
  charger's 3.0 V battery disconnect
- charge LED moved to STAT2 (charging), USB cut-off lowered to 5.4 V,
  charger /CE on a GPIO for firmware temperature control, -40 C TCXO,
  power mux on only with the amplifier, header VSYS pin removed
- firmware ceilings documented: SX1262 +20 dBm, amplifier 3.6 V by default

docs/part-audit.md: all 125 lines checked at DigiKey and LCSC (genuine
LCSC numbers, DigiKey numbers, second sources for out-of-stock lines);
parts cost about $76 at 10 boards, $58 at 100.

Schematic regenerated: ERC 0 violations, netlist equals circuit.py.

Co-Authored-By: Claude Opus 5.5 <noreply@anthropic.com>
Claude-Session: https://claude.ai/code/session_015TBB2ThqxHSgA8MkFosmn9
Parts:
- removed U9: SX1262IMLTRT, og:QFN-24_L4.0-W4.0-P0.50-BL-EP2.6, symbol og:SX1262
- added U10: SX1262IMLTRT, og:QFN-24_L4.0-W4.0-P0.50-BL-EP2.6, symbol og:SX1262
- C42: DigiKey (none) -> 1276-1067-1-ND
- C43, C44, C46: DigiKey (none) -> 1276-1001-1-ND
- C45: DigiKey (none) -> 1276-CL05A474KO5NNNCCT-ND
- C47: DigiKey (none) -> 490-3113-1-ND
- C48: DigiKey (none) -> 1276-1077-1-ND
- C49: DigiKey (none) -> 490-14446-1-ND
- C50: DigiKey (none) -> 490-8095-1-ND
- C51: DigiKey (none) -> 490-11225-1-ND
- C52: DigiKey (none) -> 490-17673-1-ND
- C53, C55: DigiKey (none) -> 490-8089-1-ND
- C54: DigiKey (none) -> 490-8093-1-ND
- L10: DigiKey (none) -> 490-1139-1-ND
- L11: DigiKey (none) -> 490-1148-1-ND
- L7: DigiKey (none) -> 445-6397-1-ND
- L8: DigiKey (none) -> 490-1154-1-ND
- L9: DigiKey (none) -> 490-6798-1-ND
- R37: DigiKey (none) -> 311-220LRCT-ND
- R38: DigiKey (none) -> 311-0.0LRCT-ND
- R39: DigiKey (none) -> 311-4.7KLRCT-ND
- R40: DigiKey (none) -> 311-10.0KLRCT-ND
- Y3: value ECS-TXO-20CSMV4-320-AY-TR -> ECS-TXO-20CSMV4-320-AP-TR; LCSC C19858587 -> C54284784; MPN ECS-TXO-20CSMV4-320-AY-TR -> ECS-TXO-20CSMV4-320-AP-TR
Connections:
- net 3V3: now also U10.1 (VDD_IN), U10.10 (VBAT), U10.11 (VBAT_IO)
- net GND: now also U10.2 (GND), U10.20 (GND), U10.25 (GND (EP)), U10.5 (GND), U10.8 (GND)
- net LORA_BUSY: now also U10.14 (BUSY)
- net LORA_DCC: now also U10.9 (DCC_SW)
- net LORA_DIO1: now also U10.13 (DIO1)
- net LORA_DIO2: now also U10.12 (DIO2)
- net LORA_DIO3: now also U10.6 (DIO3)
- net LORA_MISO: now also U10.16 (MISO)
- net LORA_MOSI: now also U10.17 (MOSI)
- net LORA_NRESET: now also U10.15 (NRESET)
- net LORA_NSS: now also U10.19 (NSS)
- net LORA_RFI_N: now also U10.22 (RFI_N)
- net LORA_RFI_P: now also U10.21 (RFI_P)
- net LORA_RFO: now also U10.23 (RFO)
- net LORA_SCK: now also U10.18 (SCK)
- net LORA_VREG: now also U10.7 (VREG)
- net LORA_VRPA: now also U10.24 (VR_PA)
- net LORA_XTA: now also U10.3 (XTA)
Changed lines of the file:
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@@
 		(on_board yes)
 		(dnp no)
-		(property "Reference" "U9"
+		(property "Reference" "U10"
 			(at 43.18 44.22 0)
 			(effects
@@
 			)
 		)
+		(property "DigiKey" "SX1262IMLTRTCT-ND"
+			(at 53.34 66.04 0)
+			(effects
+				(font
+					(size 1.27 1.27)
+				)
+				(hide yes)
+			)
+		)
 		(property "LCSC" "C191341"
 			(at 53.34 66.04 0)
@@
 			(project "mesh-radio"
 				(path "/1e0df660-60b5-6ed0-6a2a-f5098e72ebfd/d2839439-ccc6-636d-893e-761ca0d1a7fe"
-					(reference "U9")
+					(reference "U10")
 					(unit 1)
 				)
@@
 			)
 		)
-		(property "Value" "ECS-TXO-20CSMV4-320-AY-TR"
+		(property "Value" "ECS-TXO-20CSMV4-320-AP-TR"
 			(at 99.06 58.38 0)
 			(effects
@@
 			)
 		)
-		(property "MPN" "ECS-TXO-20CSMV4-320-AY-TR"
+		(property "MPN" "ECS-TXO-20CSMV4-320-AP-TR"
 			(at 104.14 50.8 0)
 			(effects
@@
 			)
 		)
-		(property "LCSC" "C19858587"
+		(property "LCSC" "C54284784"
 			(at 104.14 50.8 0)
 			(effects
@@
 			)
 		)
-		(property "Description" "TCXO 32 MHz +/-0.5 ppm, clipped sine, 2.0 x 1.6"
+		(property "Description" "TCXO 32 MHz +/-0.5 ppm, clipped sine, -40..105 C, 2.0 x 1.6 (the -AY code is only -30 C)"
 			(at 104.14 50.8 0)
 			(effects
@@
 			)
 		)
+		(property "DigiKey" "1276-1067-1-ND"
+			(at 25.4 119.38 0)
+			(effects
+				(font
+					(size 1.27 1.27)
+				)
+				(hide yes)
+			)
+		)
 		(property "LCSC" "C29266"
 			(at 25.4 119.38 0)
@@
 			)
 		)
+		(property "DigiKey" "1276-1001-1-ND"
+			(at 38.1 119.38 0)
+			(effects
+				(font
+					(size 1.27 1.27)
+				)
+				(hide yes)
+			)
+		)
 		(property "LCSC" "C1525"
 			(at 38.1 119.38 0)
@@
 			)
 		)
+		(property "DigiKey" "1276-1001-1-ND"
+			(at 50.8 119.38 0)
+			(effects
+				(font
+					(size 1.27 1.27)
+				)
+				(hide yes)
+			)
+		)
 		(property "LCSC" "C1525"
 			(at 50.8 119.38 0)
@@
 			)
 		)
+		(property "DigiKey" "1276-CL05A474KO5NNNCCT-ND"
+			(at 63.5 127 0)
+			(effects
+				(font
+					(size 1.27 1.27)
+				)
+				(hide yes)
+			)
+		)
 		(property "LCSC" "C480644"
 			(at 63.5 127 0)
@@
 			)
 		)
+		(property "DigiKey" "1276-1001-1-ND"
+			(at 76.2 127 0)
+			(effects
+				(font
+					(size 1.27 1.27)
+				)
+				(hide yes)
+			)
+		)
 		(property "LCSC" "C1525"
 			(at 76.2 127 0)
@@
 			)
 		)
+		(property "DigiKey" "1276-1077-1-ND"
+			(at 88.9 127 0)
+			(effects
+				(font
+					(size 1.27 1.27)
+				)
+				(hide yes)
+			)
+		)
 		(property "LCSC" "C307434"
 			(at 88.9 127 0)
@@
 			)
 		)
+		(property "DigiKey" "490-14446-1-ND"
+			(at 101.6 127 0)
+			(effects
+				(font
+					(size 1.27 1.27)
+				)
+				(hide yes)
+			)
+		)
 		(property "LCSC" "C161322"
 			(at 101.6 127 0)
@@
 			)
 		)
+		(property "DigiKey" "490-11225-1-ND"
+			(at 114.3 127 0)
+			(effects
+				(font
+					(size 1.27 1.27)
+				)
+				(hide yes)
+			)
+		)
 		(property "LCSC" "C161329"
 			(at 114.3 127 0)
@@
 			)
 		)
+		(property "DigiKey" "490-8089-1-ND"
+			(at 127 127 0)
+			(effects
+				(font
+					(size 1.27 1.27)
+				)
+				(hide yes)
+			)
+		)
 		(property "LCSC" "C76902"
 			(at 127 127 0)
@@
 			)
 		)
+		(property "DigiKey" "490-8089-1-ND"
+			(at 139.7 129.54 0)
+			(effects
+				(font
+					(size 1.27 1.27)
+				)
+				(hide yes)
+			)
+		)
 		(property "LCSC" "C76902"
 			(at 139.7 129.54 0)
@@
 			)
 		)
+		(property "DigiKey" "311-10.0KLRCT-ND"
+			(at 152.4 129.54 0)
+			(effects
+				(font
+					(size 1.27 1.27)
+				)
+				(hide yes)
+			)
+		)
 		(property "LCSC" "C60490"
 			(at 152.4 129.54 0)
@@
 			)
 		)
+		(property "DigiKey" "445-6397-1-ND"
+			(at 45.72 152.4 0)
+			(effects
+				(font
+					(size 1.27 1.27)
+				)
+				(hide yes)
+			)
+		)
 		(property "LCSC" "C383402"
 			(at 45.72 152.4 0)
@@
 			)
 		)
+		(property "DigiKey" "311-220LRCT-ND"
+			(at 91.44 152.4 0)
+			(effects
+				(font
+					(size 1.27 1.27)
+				)
+				(hide yes)
+			)
+		)
 		(property "LCSC" "C112291"
 			(at 91.44 152.4 0)
@@
 			)
 		)
+		(property "DigiKey" "490-3113-1-ND"
+			(at 134.62 152.4 0)
+			(effects
+				(font
+					(size 1.27 1.27)
+				)
+				(hide yes)
+			)
+		)
 		(property "LCSC" "C85874"
 			(at 134.62 152.4 0)
@@
 			)
 		)
+		(property "DigiKey" "490-1154-1-ND"
+			(at 180.34 152.4 0)
+			(effects
+				(font
+					(size 1.27 1.27)
+				)
+				(hide yes)
+			)
+		)
 		(property "LCSC" "C192855"
 			(at 180.34 152.4 0)
@@
 			)
 		)
+		(property "DigiKey" "311-0.0LRCT-ND"
+			(at 223.52 152.4 0)
+			(effects
+				(font
+					(size 1.27 1.27)
+				)
+				(hide yes)
+			)
+		)
 		(property "LCSC" "C106231"
 			(at 223.52 152.4 0)
@@
 			)
 		)
+		(property "DigiKey" "490-6798-1-ND"
+			(at 269.24 152.4 0)
+			(effects
+				(font
+					(size 1.27 1.27)
+				)
+				(hide yes)
+			)
+		)
 		(property "LCSC" "C703121"
 			(at 269.24 152.4 0)
@@
 			)
 		)
+		(property "DigiKey" "490-8095-1-ND"
+			(at 314.96 152.4 0)
+			(effects
+				(font
+					(size 1.27 1.27)
+				)
+				(hide yes)
+			)
+		)
 		(property "LCSC" "C88891"
 			(at 314.96 152.4 0)
@@
 			)
 		)
+		(property "DigiKey" "490-17673-1-ND"
+			(at 358.14 152.4 0)
+			(effects
+				(font
+					(size 1.27 1.27)
+				)
+				(hide yes)
+			)
+		)
 		(property "LCSC" "C426038"
 			(at 358.14 152.4 0)
@@
 			)
 		)
+		(property "DigiKey" "490-1139-1-ND"
+			(at 45.72 165.1 0)
+			(effects
+				(font
+					(size 1.27 1.27)
+				)
+				(hide yes)
+			)
+		)
 		(property "LCSC" "C167480"
 			(at 45.72 165.1 0)
@@
 			)
 		)
+		(property "DigiKey" "490-8093-1-ND"
+			(at 88.9 165.1 0)
+			(effects
+				(font
+					(size 1.27 1.27)
+				)
+				(hide yes)
+			)
+		)
 		(property "LCSC" "C88888"
 			(at 88.9 165.1 0)
@@
 			)
 		)
+		(property "DigiKey" "490-1148-1-ND"
+			(at 139.7 165.1 0)
+			(effects
+				(font
+					(size 1.27 1.27)
+				)
+				(hide yes)
+			)
+		)
 		(property "LCSC" "C94079"
 			(at 139.7 165.1 0)
@@
 			(at 187.96 165.1 0)
 			(effects
+				(font
+					(size 1.27 1.27)
+				)
+				(hide yes)
+			)
+		)
+		(property "DigiKey" "311-4.7KLRCT-ND"
+			(at 187.96 165.1 0)
+			(effects

Commit message: Mesh radio v1: power-path and firmware rework in progress (snapshot)
Co-Authored-By: Claude Opus 5.5 <noreply@anthropic.com>
Claude-Session: https://claude.ai/code/session_015TBB2ThqxHSgA8MkFosmn9
Parts:
- removed C54: 2.4pF, og:C_0402, symbol Device:C
- removed C55: 1.8pF, og:C_0402, symbol Device:C
- removed R37: 220R, og:R_0402, symbol Device:R
- removed R38: 0R, og:R_0402, symbol Device:R
- removed R39: 4.7k, og:R_0402, symbol Device:R
- removed R40: 10k, og:R_0402, symbol Device:R
- removed U10: SX1262IMLTRT, og:QFN-24_L4.0-W4.0-P0.50-BL-EP2.6, symbol og:SX1262
- added C40: 1uF, og:C_0402, symbol Device:C
- added C41: 100nF, og:C_0402, symbol Device:C
- added R42: 220R, og:R_0402, symbol Device:R
- added R43: 0R, og:R_0402, symbol Device:R
- added R44: 4.7k, og:R_0402, symbol Device:R
- added R45: 10k, og:R_0402, symbol Device:R
- added U9: SX1262IMLTRT, og:QFN-24_L4.0-W4.0-P0.50-BL-EP2.6, symbol og:SX1262
- C42: value 1uF -> 100nF; DigiKey 1276-1067-1-ND -> 1276-1001-1-ND; LCSC C29266 -> C1525; MPN CL05A105KO5NNNC -> CL05B104KO5NNNC
- C43: value 100nF -> 470nF; DigiKey 1276-1001-1-ND -> 1276-CL05A474KO5NNNCCT-ND; LCSC C1525 -> C480644; MPN CL05B104KO5NNNC -> CL05A474KO5NNNC
- C45: value 470nF -> 10pF; DigiKey 1276-CL05A474KO5NNNCCT-ND -> 490-3113-1-ND; LCSC C480644 -> C85874; MPN CL05A474KO5NNNC -> GJM1555C1H100JB01D; Manufacturer Samsung Electro-Mechanics -> Murata
- C46: value 100nF -> 47nF; DigiKey 1276-1001-1-ND -> 1276-1077-1-ND; LCSC C1525 -> C307434; MPN CL05B104KO5NNNC -> CL05B473KO5NNNC
- C47: value 10pF -> 47pF; DigiKey 490-3113-1-ND -> 490-14446-1-ND; LCSC C85874 -> C161322; MPN GJM1555C1H100JB01D -> GJM1555C1H470JB01D
- C48: value 47nF -> 3.0pF; DigiKey 1276-1077-1-ND -> 490-8095-1-ND; LCSC C307434 -> C88891; MPN CL05B473KO5NNNC -> GJM1555C1H3R0BB01D; Manufacturer Samsung Electro-Mechanics -> Murata
- C49: value 47pF -> 5.6pF; DigiKey 490-14446-1-ND -> 490-11225-1-ND; LCSC C161322 -> C161329; MPN GJM1555C1H470JB01D -> GJM1555C1H5R6BB01D
- C50: value 3.0pF -> 39pF; DigiKey 490-8095-1-ND -> 490-17673-1-ND; LCSC C88891 -> C426038; MPN GJM1555C1H3R0BB01D -> GJM1555C1H390JB01D
- C51: value 5.6pF -> 1.8pF; DigiKey 490-11225-1-ND -> 490-8089-1-ND; LCSC C161329 -> C76902; MPN GJM1555C1H5R6BB01D -> GJM1555C1H1R8BB01D
- C52: value 39pF -> 2.4pF; DigiKey 490-17673-1-ND -> 490-8093-1-ND; LCSC C426038 -> C88888; MPN GJM1555C1H390JB01D -> GJM1555C1H2R4BB01D
Connections:
- net 3V3: now also C40.1, C41.1, U9.1 (VDD_IN), U9.10 (VBAT), U9.11 (VBAT_IO); no longer C43.1, C44.1
- net GND: now also C47.2, C40.2, C41.2, R45.2, U9.2 (GND), U9.20 (GND), U9.25 (GND (EP)), U9.5 (GND), U9.8 (GND); no longer C45.2, C48.2
- net LNA_OUT: now also C52.1
- net LORA_BUSY: now also U9.14 (BUSY)
- net LORA_DCC: now also U9.9 (DCC_SW)
- net LORA_DIO1: now also U9.13 (DIO1)
- net LORA_DIO2: now also R44.1, U9.12 (DIO2)
- net LORA_DIO3: now also C44.1, U9.6 (DIO3); no longer C46.1
- net LORA_MISO: now also U9.16 (MISO)
- net LORA_MOSI: now also U9.17 (MOSI)
- net LORA_NRESET: now also U9.15 (NRESET)
- net LORA_NSS: now also U9.19 (NSS)
- net LORA_RFI_N: now also C52.2, U9.22 (RFI_N)
- net LORA_RFI_P: now also C53.1, U9.21 (RFI_P)
- net LORA_RFO: now also R43.1, U9.23 (RFO)
- net LORA_SCK: now also U9.18 (SCK)
- net LORA_TX50: now also C51.1; no longer C53.1
- net LORA_TXA: now also C48.1, R43.2; no longer C50.1
- net LORA_TXB: now also C48.2, C49.1, C50.1; no longer C50.2, C51.1, C52.1
- net LORA_TXC: now also C50.2; no longer C52.2
- net LORA_VREG: now also C43.1, U9.7 (VREG); no longer C45.1
- net LORA_VRPA: now also C46.1, C47.1, U9.24 (VR_PA); no longer C48.1, C49.1
- net LORA_XTA: now also C45.2, U9.3 (XTA); no longer C47.2
- net RF_SW_CTRL: now also R44.2, R45.1
- net TCXO_AC: now also C45.1, R42.2; no longer C47.1
- net TCXO_OUT: now also R42.1
Other:
- moved on the sheet: C42, C43, C44, C45, C46, C47, C48, C49, C50, C51, C52, C53
Changed lines of the file:
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@@
 		(on_board yes)
 		(dnp no)
-		(property "Reference" "U10"
+		(property "Reference" "U9"
 			(at 43.18 44.22 0)
 			(effects
@@
 			(project "mesh-radio"
 				(path "/1e0df660-60b5-6ed0-6a2a-f5098e72ebfd/d2839439-ccc6-636d-893e-761ca0d1a7fe"
-					(reference "U10")
+					(reference "U9")
 					(unit 1)
 				)
@@
 		(on_board yes)
 		(dnp no)
-		(property "Reference" "C42"
+		(property "Reference" "C40"
 			(at 27.2 118.38 0)
 			(effects
@@
 			(project "mesh-radio"
 				(path "/1e0df660-60b5-6ed0-6a2a-f5098e72ebfd/d2839439-ccc6-636d-893e-761ca0d1a7fe"
-					(reference "C42")
+					(reference "C40")
 					(unit 1)
 				)
@@
 		(on_board yes)
 		(dnp no)
-		(property "Reference" "C43"
+		(property "Reference" "C41"
 			(at 39.9 118.38 0)
 			(effects
@@
 			(project "mesh-radio"
 				(path "/1e0df660-60b5-6ed0-6a2a-f5098e72ebfd/d2839439-ccc6-636d-893e-761ca0d1a7fe"
-					(reference "C43")
+					(reference "C41")
 					(unit 1)
 				)
@@
 		(on_board yes)
 		(dnp no)
-		(property "Reference" "C44"
+		(property "Reference" "C42"
 			(at 52.6 118.38 0)
 			(effects
@@
 			(project "mesh-radio"
 				(path "/1e0df660-60b5-6ed0-6a2a-f5098e72ebfd/d2839439-ccc6-636d-893e-761ca0d1a7fe"
-					(reference "C44")
+					(reference "C42")
 					(unit 1)
 				)
@@
 		(on_board yes)
 		(dnp no)
-		(property "Reference" "C45"
+		(property "Reference" "C43"
 			(at 65.3 126 0)
 			(effects
@@
 			(project "mesh-radio"
 				(path "/1e0df660-60b5-6ed0-6a2a-f5098e72ebfd/d2839439-ccc6-636d-893e-761ca0d1a7fe"
-					(reference "C45")
+					(reference "C43")
 					(unit 1)
 				)
@@
 		(on_board yes)
 		(dnp no)
-		(property "Reference" "C46"
+		(property "Reference" "C44"
 			(at 78 126 0)
 			(effects
@@
 			(project "mesh-radio"
 				(path "/1e0df660-60b5-6ed0-6a2a-f5098e72ebfd/d2839439-ccc6-636d-893e-761ca0d1a7fe"
-					(reference "C46")
+					(reference "C44")
 					(unit 1)
 				)
@@
 		(on_board yes)
 		(dnp no)
-		(property "Reference" "C48"
+		(property "Reference" "C46"
 			(at 90.7 126 0)
 			(effects
@@
 			(project "mesh-radio"
 				(path "/1e0df660-60b5-6ed0-6a2a-f5098e72ebfd/d2839439-ccc6-636d-893e-761ca0d1a7fe"
-					(reference "C48")
+					(reference "C46")
 					(unit 1)
 				)
@@
 		(on_board yes)
 		(dnp no)
-		(property "Reference" "C49"
+		(property "Reference" "C47"
 			(at 103.4 126 0)
 			(effects
@@
 			(project "mesh-radio"
 				(path "/1e0df660-60b5-6ed0-6a2a-f5098e72ebfd/d2839439-ccc6-636d-893e-761ca0d1a7fe"
-					(reference "C49")
+					(reference "C47")
 					(unit 1)
 				)
@@
 		(on_board yes)
 		(dnp no)
-		(property "Reference" "C51"
+		(property "Reference" "C49"
 			(at 116.1 126 0)
 			(effects
@@
 			(project "mesh-radio"
 				(path "/1e0df660-60b5-6ed0-6a2a-f5098e72ebfd/d2839439-ccc6-636d-893e-761ca0d1a7fe"
-					(reference "C51")
+					(reference "C49")
 					(unit 1)
 				)
@@
 		(on_board yes)
 		(dnp no)
-		(property "Reference" "C53"
+		(property "Reference" "C51"
 			(at 128.8 126 0)
 			(effects
@@
 			(project "mesh-radio"
 				(path "/1e0df660-60b5-6ed0-6a2a-f5098e72ebfd/d2839439-ccc6-636d-893e-761ca0d1a7fe"
-					(reference "C53")
+					(reference "C51")
 					(unit 1)
 				)
@@
 		(on_board yes)
 		(dnp no)
-		(property "Reference" "C55"
+		(property "Reference" "C53"
 			(at 141.5 128.54 0)
 			(effects
@@
 			(project "mesh-radio"
 				(path "/1e0df660-60b5-6ed0-6a2a-f5098e72ebfd/d2839439-ccc6-636d-893e-761ca0d1a7fe"
-					(reference "C55")
+					(reference "C53")
 					(unit 1)
 				)
@@
 		(on_board yes)
 		(dnp no)
-		(property "Reference" "R40"
+		(property "Reference" "R45"
 			(at 154.2 128.54 0)
 			(effects
@@
 			(project "mesh-radio"
 				(path "/1e0df660-60b5-6ed0-6a2a-f5098e72ebfd/d2839439-ccc6-636d-893e-761ca0d1a7fe"
-					(reference "R40")
+					(reference "R45")
 					(unit 1)
 				)
@@
 		(on_board yes)
 		(dnp no)
-		(property "Reference" "R37"
+		(property "Reference" "R42"
 			(at 91.44 149.8 0)
 			(effects
@@
 			(project "mesh-radio"
 				(path "/1e0df660-60b5-6ed0-6a2a-f5098e72ebfd/d2839439-ccc6-636d-893e-761ca0d1a7fe"
-					(reference "R37")
+					(reference "R42")
 					(unit 1)
 				)
@@
 		(on_board yes)
 		(dnp no)
-		(property "Reference" "C47"
+		(property "Reference" "C45"
 			(at 134.62 149.8 0)
 			(effects
@@
 			(project "mesh-radio"
 				(path "/1e0df660-60b5-6ed0-6a2a-f5098e72ebfd/d2839439-ccc6-636d-893e-761ca0d1a7fe"
-					(reference "C47")
+					(reference "C45")
 					(unit 1)
 				)
@@
 		(on_board yes)
 		(dnp no)
-		(property "Reference" "R38"
+		(property "Reference" "R43"
 			(at 223.52 149.8 0)
 			(effects
@@
 			(project "mesh-radio"
 				(path "/1e0df660-60b5-6ed0-6a2a-f5098e72ebfd/d2839439-ccc6-636d-893e-761ca0d1a7fe"
-					(reference "R38")
+					(reference "R43")
 					(unit 1)
 				)
@@
 		(on_board yes)
 		(dnp no)
-		(property "Reference" "C50"
+		(property "Reference" "C48"
 			(at 314.96 149.8 0)
 			(effects
@@
 			(project "mesh-radio"
 				(path "/1e0df660-60b5-6ed0-6a2a-f5098e72ebfd/d2839439-ccc6-636d-893e-761ca0d1a7fe"
-					(reference "C50")
+					(reference "C48")
 					(unit 1)
 				)
@@
 		(on_board yes)
 		(dnp no)
-		(property "Reference" "C52"
+		(property "Reference" "C50"
 			(at 358.14 149.8 0)
 			(effects
@@
 			(project "mesh-radio"
 				(path "/1e0df660-60b5-6ed0-6a2a-f5098e72ebfd/d2839439-ccc6-636d-893e-761ca0d1a7fe"
-					(reference "C52")
+					(reference "C50")
 					(unit 1)
 				)
@@
 		(on_board yes)
 		(dnp no)
-		(property "Reference" "C54"
+		(property "Reference" "C52"
 			(at 88.9 162.5 0)
 			(effects
@@
 			(project "mesh-radio"
 				(path "/1e0df660-60b5-6ed0-6a2a-f5098e72ebfd/d2839439-ccc6-636d-893e-761ca0d1a7fe"
-					(reference "C54")
+					(reference "C52")
 					(unit 1)
 				)
@@
 		(on_board yes)
 		(dnp no)
-		(property "Reference" "R39"
+		(property "Reference" "R44"
 			(at 187.96 162.5 0)
 			(effects
@@
 			(project "mesh-radio"
 				(path "/1e0df660-60b5-6ed0-6a2a-f5098e72ebfd/d2839439-ccc6-636d-893e-761ca0d1a7fe"
-					(reference "R39")
+					(reference "R44")
 					(unit 1)
 				)

Commit message: Mesh Radio v1 schematic: regenerated (gate clamp, NTC part); ERC 0, netlist equal
Co-Authored-By: Claude Opus 5.5 <noreply@anthropic.com>
Claude-Session: https://claude.ai/code/session_015TBB2ThqxHSgA8MkFosmn9
Parts:
- Y3: DigiKey (none) -> 50-ECS-TXO-20CSMV4-320-AP-TRCT-ND
Changed lines of the file:
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@@
+			)
+		)
+		(property "DigiKey" "50-ECS-TXO-20CSMV4-320-AP-TRCT-ND"
+			(at 104.14 50.8 0)
+			(effects
+				(font
+					(size 1.27 1.27)
+				)
+				(hide yes)
 			)
 		)
