File: mesh-radio/v1/schematic/ports.kicad_sch (KiCad schematic)
At the start: 22 parts, among them J5 SM06B-GHS-TB(LF)(SN), J6 SM06B-SRSS-TB(LF)(SN), J7 EXPANSION, SW2 B3U-1000P, SW3 B3U-1000P, U17 TPS22916CYFPR

Commit message: Mesh Radio v1: fix every design-review finding, add the part audit
An independent review of the schematic found two critical and nine further
issues; all are fixed in src/circuit.py:
- reverse-battery FET gate now returns to the cell's own minus terminal, so
  a backwards cell stays isolated even while USB/solar/drone power the board
- solar and drone inputs: reverse-blocking Schottky + 22 V flat-clamp TVS
  (the 15 V TVS would have failed on a 12 V panel); 4.7 V clamp on every
  eFuse EN/UVLO pin so 20 V on an input stays inside its rating
- ideal diode (LM66100) holds VSYS on the cell when a 3 W burst trips the
  charger's 3.0 V battery disconnect
- charge LED moved to STAT2 (charging), USB cut-off lowered to 5.4 V,
  charger /CE on a GPIO for firmware temperature control, -40 C TCXO,
  power mux on only with the amplifier, header VSYS pin removed
- firmware ceilings documented: SX1262 +20 dBm, amplifier 3.6 V by default

docs/part-audit.md: all 125 lines checked at DigiKey and LCSC (genuine
LCSC numbers, DigiKey numbers, second sources for out-of-stock lines);
parts cost about $76 at 10 boards, $58 at 100.

Schematic regenerated: ERC 0 violations, netlist equals circuit.py.

Co-Authored-By: Claude Opus 5.5 <noreply@anthropic.com>
Claude-Session: https://claude.ai/code/session_015TBB2ThqxHSgA8MkFosmn9
Parts:
- removed D6, D7: TPD4E05U06DQAR, og:USON-10_L2.5-W1.0-P0.50-BL, symbol og:TPD4E05U06
- removed U17: TPS22916CYFPR, og:DSBGA-4_TPS22916, symbol og:TPS22916
- added D11, D12: TPD4E05U06DQAR, og:USON-10_L2.5-W1.0-P0.50-BL, symbol og:TPD4E05U06
- added U18: TPS22916CYFPR, og:DSBGA-4_TPS22916, symbol og:TPS22916
- C99: DigiKey (none) -> 1276-1067-1-ND
- J5: DigiKey (none) -> 455-1568-1-ND
- J6: DigiKey (none) -> 455-SM06B-SRSS-TBCT-ND
- LED2: DigiKey (none) -> 160-1446-1-ND
- LED3: DigiKey (none) -> 160-1647-1-ND
- R56, R57, R58, R59, R60, R61, R62, R63: DigiKey (none) -> 311-470LRCT-ND
- R64: DigiKey (none) -> 311-1.00MLRCT-ND
- R65: DigiKey (none) -> 311-1.00KLRCT-ND
- R66: value 1k -> 220R; DigiKey (none) -> 311-220LRCT-ND; LCSC C106235 -> C112291; MPN RC0402FR-071KL -> RC0402FR-07220RL
- SW2, SW3: DigiKey (none) -> SW1020CT-ND
Connections:
- net VSYS_SW is gone; now on net GND: J7.18
- net 3V3: now also U18.A2 (VIN)
- net 3V3_GPS: now also U18.A1 (VOUT)
- net DRN_P2: now also D11.1 (IO1)
- net DRN_P3: now also D11.2 (IO2)
- net DRN_P4: now also D11.4 (IO3)
- net DRN_P5: now also D11.5 (IO4)
- net GND: now also D11.3 (GND), D11.8 (GND), D12.3 (GND), D12.8 (GND), U18.B1 (GND)
- net GPS_EN: now also U18.B2 (ON)
- net GPS_P2: now also D12.1 (IO1)
- net GPS_P3: now also D12.2 (IO2)
- net GPS_P4: now also D12.4 (IO3)
- net GPS_P5: now also D12.5 (IO4)
- net DRONE_5V_RAW renamed DRONE_5V_CONN
Other:
- moved on the sheet: J6, J7

Commit message: Mesh radio v1: build on KiCad 10.0.7 (latest stable, 7 Oct 2026)
The toolchain image now starts from kicad/kicad:10.0.7, pinned by digest.
Rebuilt on it: the schematic (ERC 0, netlist equals circuit.py) and the
placed board (DRC 0).  The regenerated schematic also picks up the
expansion header's current footprint (og:Header_2x1x10_Rows20.32), which
the committed sheet still named by its old one.

Co-Authored-By: Claude Opus 5.5 <noreply@anthropic.com>
Claude-Session: https://claude.ai/code/session_015TBB2ThqxHSgA8MkFosmn9
Parts:
- J7: footprint og:PinHeader_2x10_P2.54mm -> og:Header_2x1x10_Rows20.32
Changed lines of the file:
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@@
 			)
 		)
-		(property "Footprint" "og:PinHeader_2x10_P2.54mm"
+		(property "Footprint" "og:Header_2x1x10_Rows20.32"
 			(at 256.54 60.96 0)
 			(effects

Commit message: Mesh radio v1: LFCG-1000+ antenna filter; missing-antenna detector
Owner decisions of 19 Oct: keep 3 W with the heat fixes and a gap pad to
a metal enclosure, 6 layers, 300 mA charging, new parts at the designer's
judgement.  This commit, from sim/rf:
- FL1 LFCN-1000+ (1206) -> LFCG-1000+ (0805, 8 pads, Mini-Circuits case
  GE0805C-2: in 8, out 4): no stop-band re-entry at 5.5-10 GHz, where the
  3 W 6th-10th harmonics failed FCC's restricted-band limit;
- a reflected-wave detector: a printed line beside the ANT line
  terminated in 49.9 R, an Infineon BAT15-02EL, 1 nF and 100 k into
  P0.30/AIN6, so firmware can cut the amplifier within ~1 ms of a packet
  with no antenna (the antenna switch sees 109-160 % of its rating then);
- P0.31/AIN7 reads the charger's NTC (firmware's 0-45 C charging rule);
  the expansion header's IO3/IO4 give way (four spare pins remain).
ERC 0, netlist equals circuit.py, every pin and pad accounted for.

Co-Authored-By: Claude Opus 5.5 <noreply@anthropic.com>
Claude-Session: https://claude.ai/code/session_015TBB2ThqxHSgA8MkFosmn9
Parts:
- removed C99: 1uF, og:C_0402, symbol Device:C
- removed D11: TPD4E05U06DQAR, og:USON-10_L2.5-W1.0-P0.50-BL, symbol og:TPD4E05U06
- removed R56, R57: 470R, og:R_0402, symbol Device:R
- added C100: 1uF, og:C_0402, symbol Device:C
- added D13: TPD4E05U06DQAR, og:USON-10_L2.5-W1.0-P0.50-BL, symbol og:TPD4E05U06
- added R67: 1k, og:R_0402, symbol Device:R
- added R68: 220R, og:R_0402, symbol Device:R
- R64: value 1M -> 470R; DigiKey 311-1.00MLRCT-ND -> 311-470LRCT-ND; LCSC C138033 -> C114877; MPN RC0402FR-071ML -> RC0402FR-07470RL
- R65: value 1k -> 470R; DigiKey 311-1.00KLRCT-ND -> 311-470LRCT-ND; LCSC C106235 -> C114877; MPN RC0402FR-071KL -> RC0402FR-07470RL
- R66: value 220R -> 1M; DigiKey 311-220LRCT-ND -> 311-1.00MLRCT-ND; LCSC C112291 -> C138033; MPN RC0402FR-07220RL -> RC0402FR-071ML
Connections:
- net 3V3_GPS: now also C100.1
- net DRN_P2: now also D12.1 (IO1), R58.1
- net DRN_P3: now also D12.2 (IO2), R59.2
- net DRN_P4: now also D12.4 (IO3), R60.2; no longer R58.2
- net DRN_P5: now also D12.5 (IO4), R61.1; no longer R59.1
- net DRONE_CTS: now also R61.2; no longer R59.2
- net DRONE_RTS: now also R60.1; no longer R58.1
- net DRONE_RX: now also R58.2
- net DRONE_TX: now also R59.1
- net GND: now also R66.2, C100.2, D13.3 (GND), D13.8 (GND); no longer R64.2
- net GPS_EN: now also R66.1; no longer R64.1
- net GPS_P2: now also R62.1, D13.1 (IO1); no longer D12.1 (IO1), R60.1
- net GPS_P3: now also R63.2, D13.2 (IO2); no longer D12.2 (IO2), R61.2
- net GPS_P4: now also R64.1, D13.4 (IO3); no longer D12.4 (IO3), R62.1
- net GPS_P5: now also R65.2, D13.5 (IO4); no longer D12.5 (IO4), R63.2
- net GPS_PPS: now also R64.2; no longer R62.2
- net GPS_RESET: now also R65.1; no longer R63.1
- net GPS_RX: now also R62.2; no longer R60.2
- net GPS_TX: now also R63.1; no longer R61.1
- net LED_BLUE: now also R68.1; no longer R66.1
- net LED_B_A: now also R68.2; no longer R66.2
- net LED_GREEN: now also R67.1; no longer R65.1
- net LED_G_A: now also R67.2; no longer R65.2
- net IO3: no longer names the net of J7.14
- net IO4: no longer names the net of J7.15
- no-connect marks 12 -> 14
Other:
- moved on the sheet: D12, R58, R59, R60, R61, R62, R63, R64, R65, R66
Changed lines of the file:
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@@
 		(on_board yes)
 		(dnp no)
-		(property "Reference" "D11"
+		(property "Reference" "D12"
 			(at 88.9 44.22 0)
 			(effects
@@
 			(project "mesh-radio"
 				(path "/1e0df660-60b5-6ed0-6a2a-f5098e72ebfd/7f4f5fdb-9d3f-986c-3228-336ce6b7a0b3"
-					(reference "D11")
+					(reference "D12")
 					(unit 1)
 				)
@@
 		(on_board yes)
 		(dnp no)
-		(property "Reference" "D12"
+		(property "Reference" "D13"
 			(at 167.64 44.22 0)
 			(effects
@@
 			(project "mesh-radio"
 				(path "/1e0df660-60b5-6ed0-6a2a-f5098e72ebfd/7f4f5fdb-9d3f-986c-3228-336ce6b7a0b3"
-					(reference "D12")
+					(reference "D13")
 					(unit 1)
 				)
@@
 		)
 	)
-	(wire
-		(pts
-			(xy 248.92 66.04)
-			(xy 246.38 66.04)
-		)
-		(stroke
-			(width 0)
-			(type default)
-		)
-	)
-	(global_label "IO4"
-		(shape passive)
-		(at 246.38 66.04 180)
-		(fields_autoplaced yes)
-		(effects
-			(font
-				(size 1.27 1.27)
-			)
-			(justify right)
-		)
-		(property "Intersheetrefs" "${INTERSHEET_REFS}"
-			(at 246.38 66.04 0)
-			(effects
-				(font
-					(size 1.27 1.27)
-				)
-				(justify right)
-				(hide yes)
-			)
-		)
+	(no_connect
+		(at 248.92 66.04)
 	)
 	(wire
@@
 		)
 	)
-	(wire
-		(pts
-			(xy 264.16 63.5)
-			(xy 266.7 63.5)
-		)
-		(stroke
-			(width 0)
-			(type default)
-		)
-	)
-	(global_label "IO3"
-		(shape passive)
-		(at 266.7 63.5 0)
-		(fields_autoplaced yes)
-		(effects
-			(font
-				(size 1.27 1.27)
-			)
-			(justify left)
-		)
-		(property "Intersheetrefs" "${INTERSHEET_REFS}"
-			(at 266.7 63.5 0)
-			(effects
-				(font
-					(size 1.27 1.27)
-				)
-				(justify left)
-				(hide yes)
-			)
-		)
+	(no_connect
+		(at 264.16 63.5)
 	)
 	(wire
@@
 		(on_board yes)
 		(dnp no)
-		(property "Reference" "R64"
+		(property "Reference" "R66"
 			(at 27.2 110.76 0)
 			(effects
@@
 			(project "mesh-radio"
 				(path "/1e0df660-60b5-6ed0-6a2a-f5098e72ebfd/7f4f5fdb-9d3f-986c-3228-336ce6b7a0b3"
-					(reference "R64")
+					(reference "R66")
 					(unit 1)
 				)
@@
 		(on_board yes)
 		(dnp no)
-		(property "Reference" "C99"
+		(property "Reference" "C100"
 			(at 39.9 105.68 0)
 			(effects
@@
 			(project "mesh-radio"
 				(path "/1e0df660-60b5-6ed0-6a2a-f5098e72ebfd/7f4f5fdb-9d3f-986c-3228-336ce6b7a0b3"
-					(reference "C99")
+					(reference "C100")
 					(unit 1)
 				)
@@
 		(on_board yes)
 		(dnp no)
-		(property "Reference" "R56"
+		(property "Reference" "R58"
 			(at 43.18 134.56 0)
 			(effects
@@
 			(project "mesh-radio"
 				(path "/1e0df660-60b5-6ed0-6a2a-f5098e72ebfd/7f4f5fdb-9d3f-986c-3228-336ce6b7a0b3"
-					(reference "R56")
+					(reference "R58")
 					(unit 1)
 				)
@@
 		(on_board yes)
 		(dnp no)
-		(property "Reference" "R57"
+		(property "Reference" "R59"
 			(at 88.9 134.56 0)
 			(effects
@@
 			(project "mesh-radio"
 				(path "/1e0df660-60b5-6ed0-6a2a-f5098e72ebfd/7f4f5fdb-9d3f-986c-3228-336ce6b7a0b3"
-					(reference "R57")
+					(reference "R59")
 					(unit 1)
 				)
@@
 		(on_board yes)
 		(dnp no)
-		(property "Reference" "R58"
+		(property "Reference" "R60"
 			(at 132.08 134.56 0)
 			(effects
@@
 			(project "mesh-radio"
 				(path "/1e0df660-60b5-6ed0-6a2a-f5098e72ebfd/7f4f5fdb-9d3f-986c-3228-336ce6b7a0b3"
-					(reference "R58")
+					(reference "R60")
 					(unit 1)
 				)
@@
 		(on_board yes)
 		(dnp no)
-		(property "Reference" "R59"
+		(property "Reference" "R61"
 			(at 172.72 134.56 0)
 			(effects
@@
 			(project "mesh-radio"
 				(path "/1e0df660-60b5-6ed0-6a2a-f5098e72ebfd/7f4f5fdb-9d3f-986c-3228-336ce6b7a0b3"
-					(reference "R59")
+					(reference "R61")
 					(unit 1)
 				)
@@
 		(on_board yes)
 		(dnp no)
-		(property "Reference" "R60"
+		(property "Reference" "R62"
 			(at 215.9 134.56 0)
 			(effects
@@
 			(project "mesh-radio"
 				(path "/1e0df660-60b5-6ed0-6a2a-f5098e72ebfd/7f4f5fdb-9d3f-986c-3228-336ce6b7a0b3"
-					(reference "R60")
+					(reference "R62")
 					(unit 1)
 				)
@@
 		(on_board yes)
 		(dnp no)
-		(property "Reference" "R61"
+		(property "Reference" "R63"
 			(at 256.54 134.56 0)
 			(effects
@@
 			(project "mesh-radio"
 				(path "/1e0df660-60b5-6ed0-6a2a-f5098e72ebfd/7f4f5fdb-9d3f-986c-3228-336ce6b7a0b3"
-					(reference "R61")
+					(reference "R63")
 					(unit 1)
 				)
@@
 		(on_board yes)
 		(dnp no)
-		(property "Reference" "R62"
+		(property "Reference" "R64"
 			(at 299.72 134.56 0)
 			(effects
@@
 			(project "mesh-radio"
 				(path "/1e0df660-60b5-6ed0-6a2a-f5098e72ebfd/7f4f5fdb-9d3f-986c-3228-336ce6b7a0b3"
-					(reference "R62")
+					(reference "R64")
 					(unit 1)
 				)
@@
 		(on_board yes)
 		(dnp no)
-		(property "Reference" "R63"
+		(property "Reference" "R65"
 			(at 342.9 134.56 0)
 			(effects
@@
 			(project "mesh-radio"
 				(path "/1e0df660-60b5-6ed0-6a2a-f5098e72ebfd/7f4f5fdb-9d3f-986c-3228-336ce6b7a0b3"
-					(reference "R63")
+					(reference "R65")
 					(unit 1)
 				)
@@
 		(on_board yes)
 		(dnp no)
-		(property "Reference" "R65"
+		(property "Reference" "R67"
 			(at 45.72 147.26 0)
 			(effects
@@
 			(project "mesh-radio"
 				(path "/1e0df660-60b5-6ed0-6a2a-f5098e72ebfd/7f4f5fdb-9d3f-986c-3228-336ce6b7a0b3"
-					(reference "R65")
+					(reference "R67")
 					(unit 1)
 				)
@@
 		(on_board yes)
 		(dnp no)
-		(property "Reference" "R66"
+		(property "Reference" "R68"
 			(at 88.9 147.26 0)
 			(effects
@@
 			(project "mesh-radio"
 				(path "/1e0df660-60b5-6ed0-6a2a-f5098e72ebfd/7f4f5fdb-9d3f-986c-3228-336ce6b7a0b3"
-					(reference "R66")
+					(reference "R68")
 					(unit 1)
 				)

Commit message: Mesh radio v1: power-path and firmware rework in progress (snapshot)
Co-Authored-By: Claude Opus 5.5 <noreply@anthropic.com>
Claude-Session: https://claude.ai/code/session_015TBB2ThqxHSgA8MkFosmn9
Parts:
- removed C100: 1uF, og:C_0402, symbol Device:C
- removed D12, D13: TPD4E05U06DQAR, og:USON-10_L2.5-W1.0-P0.50-BL, symbol og:TPD4E05U06
- removed R58, R59, R60, R61, R62: 470R, og:R_0402, symbol Device:R
- removed U18: TPS22916CYFPR, og:DSBGA-4_TPS22916, symbol og:TPS22916
- added C98: 1uF, og:C_0402, symbol Device:C
- added D10, D9: TPD4E05U06DQAR, og:USON-10_L2.5-W1.0-P0.50-BL, symbol og:TPD4E05U06
- added R69, R70: 470R, og:R_0402, symbol Device:R
- added R71: 1M, og:R_0402, symbol Device:R
- added R72: 1k, og:R_0402, symbol Device:R
- added R73: 220R, og:R_0402, symbol Device:R
- added U17: TPS22916CYFPR, og:DSBGA-4_TPS22916, symbol og:TPS22916
- R66: value 1M -> 470R; DigiKey 311-1.00MLRCT-ND -> 311-470LRCT-ND; LCSC C138033 -> C114877; MPN RC0402FR-071ML -> RC0402FR-07470RL
- R67: value 1k -> 470R; DigiKey 311-1.00KLRCT-ND -> 311-470LRCT-ND; LCSC C106235 -> C114877; MPN RC0402FR-071KL -> RC0402FR-07470RL
- R68: value 220R -> 470R; DigiKey 311-220LRCT-ND -> 311-470LRCT-ND; LCSC C112291 -> C114877; MPN RC0402FR-07220RL -> RC0402FR-07470RL
- SW2, SW3: value B3U-1000P -> SKRPADE010; footprint og:KEY-SMD_B3U-1000PM -> og:KEY-SMD_4P-L4.2-W3.2-P2.20-LS4.6; symbol Switch:SW_Push -> og:SKRP; DigiKey SW1020CT-ND -> 4809-SKRPADE010CT-ND; LCSC C231329 -> C127488; MPN B3U-1000P -> SKRPADE010; Manufacturer Omron (Aratas) -> Alps Alpine
Connections:
- net 3V3: now also U17.A2 (VIN)
- net 3V3_GPS: now also C98.1, U17.A1 (VOUT)
- net BTN_USER: now also SW3.2 (A)
- net DRN_P2: now also R63.1, D9.1 (IO1)
- net DRN_P3: now also R64.2, D9.2 (IO2)
- net DRN_P4: now also R65.2, D9.4 (IO3)
- net DRN_P5: now also R66.1, D9.5 (IO4)
- net DRONE_CTS: now also R66.2
- net DRONE_RTS: now also R65.1
- net DRONE_RX: now also R63.2
- net DRONE_TX: now also R64.1
- net GND: now also SW2.3 (B), SW2.4 (B), SW3.3 (B), SW3.4 (B), C98.2, D10.3 (GND), D10.8 (GND), D9.3 (GND), D9.8 (GND), R71.2, U17.B1 (GND); no longer R66.2, SW2.2, SW3.2
- net GPS_EN: now also R71.1, U17.B2 (ON); no longer R66.1
- net GPS_P2: now also R67.1, D10.1 (IO1)
- net GPS_P3: now also R68.2, D10.2 (IO2); no longer R63.2
- net GPS_P4: now also D10.4 (IO3), R69.1; no longer R64.1
- net GPS_P5: now also D10.5 (IO4), R70.2; no longer R65.2
- net GPS_PPS: now also R69.2; no longer R64.2
- net GPS_RESET: now also R70.1; no longer R65.1
- net GPS_RX: now also R67.2
- net GPS_TX: now also R68.1; no longer R63.1
- net LED_BLUE: now also R73.1; no longer R68.1
- net LED_B_A: now also R73.2; no longer R68.2
- net LED_GREEN: now also R72.1; no longer R67.1
- net LED_G_A: now also R72.2; no longer R67.2
- net NRF_RESET: now also SW2.2 (A)
Other:
- moved on the sheet: LED2, LED3, R63, R64, R65, R66, R67, R68

Commit message: Mesh Radio v1 schematic: regenerated (gate clamp, NTC part); ERC 0, netlist equal
Co-Authored-By: Claude Opus 5.5 <noreply@anthropic.com>
Claude-Session: https://claude.ai/code/session_015TBB2ThqxHSgA8MkFosmn9
Parts:
- removed D9: TPD4E05U06DQAR, og:USON-10_L2.5-W1.0-P0.50-BL, symbol og:TPD4E05U06
- added D11: TPD4E05U06DQAR, og:USON-10_L2.5-W1.0-P0.50-BL, symbol og:TPD4E05U06
Connections:
- net DRN_P2: now also D10.1 (IO1)
- net DRN_P3: now also D10.2 (IO2)
- net DRN_P4: now also D10.4 (IO3)
- net DRN_P5: now also D10.5 (IO4)
- net GND: now also D11.3 (GND), D11.8 (GND)
- net GPS_P2: now also D11.1 (IO1); no longer D10.1 (IO1)
- net GPS_P3: now also D11.2 (IO2); no longer D10.2 (IO2)
- net GPS_P4: now also D11.4 (IO3); no longer D10.4 (IO3)
- net GPS_P5: now also D11.5 (IO4); no longer D10.5 (IO4)
Other:
- moved on the sheet: D10
Changed lines of the file:
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@@
 		(on_board yes)
 		(dnp no)
-		(property "Reference" "D9"
+		(property "Reference" "D10"
 			(at 88.9 44.22 0)
 			(effects
@@
 			(project "mesh-radio"
 				(path "/1e0df660-60b5-6ed0-6a2a-f5098e72ebfd/7f4f5fdb-9d3f-986c-3228-336ce6b7a0b3"
-					(reference "D9")
+					(reference "D10")
 					(unit 1)
 				)
@@
 		(on_board yes)
 		(dnp no)
-		(property "Reference" "D10"
+		(property "Reference" "D11"
 			(at 167.64 44.22 0)
 			(effects
@@
 			(project "mesh-radio"
 				(path "/1e0df660-60b5-6ed0-6a2a-f5098e72ebfd/7f4f5fdb-9d3f-986c-3228-336ce6b7a0b3"
-					(reference "D10")
+					(reference "D11")
 					(unit 1)
 				)

Commit message: Mesh Radio v1: ratio detector circuit and RF re-run in progress (snapshot)
Co-Authored-By: Claude Opus 5.5 <noreply@anthropic.com>
Claude-Session: https://claude.ai/code/session_015TBB2ThqxHSgA8MkFosmn9
Parts:
- R70: value 470R -> 100k; DigiKey 311-470LRCT-ND -> 311-100KLRCT-ND; LCSC C114877 -> C60491; MPN RC0402FR-07470RL -> RC0402FR-07100KL
Connections:
- net GPS_RESET is gone; now on net GPS_P5: R70.1
- net 3V3_GPS: now also R70.2
- net GPS_P5: no longer R70.2
Other:
- moved on the sheet: C98, LED2, LED3, R70, R71, R72, R73
