File: mesh-radio/v1/schematic/frontend.kicad_sch (KiCad schematic)
At the start: 59 parts, among them J4 U.FL-R-SMT-1(80), U10 QPA9510TR7, U11 SKY13330-397LF, U12 BGA7L1BN6E6327XTSA1

Commit message: Mesh Radio v1: detector placed (diodes at the coupled line's ends, caps beside)
The reflected diode stands straight above the U.FL-end 49.9 R, turned
so the line meets only its anode; the forward diode sits at the filter
end on the line's level. The U.FL-end 49.9 R is an 0402 (21 mW, 40 % of
its 85 C rating) to fit beside the U.FL. Schematic regenerated.

Co-Authored-By: Claude Opus 5.5 <noreply@anthropic.com>
Claude-Session: https://claude.ai/code/session_015TBB2ThqxHSgA8MkFosmn9
Parts:
- R75: footprint og:R_0805 -> og:R_0402; DigiKey 541-49.9TCT-ND -> 311-49.9LRCT-ND; LCSC C4088942 -> C87044; MPN CRCW080549R9FKEAHP -> RC0402FR-0749R9L; Manufacturer Vishay Dale -> Yageo
Changed lines of the file:
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@@
 			)
 		)
-		(property "Footprint" "og:R_0805"
+		(property "Footprint" "og:R_0402"
 			(at 165.1 157.48 0)
 			(effects
@@
 			)
 		)
-		(property "MPN" "CRCW080549R9FKEAHP"
+		(property "MPN" "RC0402FR-0749R9L"
 			(at 165.1 157.48 0)
 			(effects
@@
 			)
 		)
-		(property "Manufacturer" "Vishay Dale"
+		(property "Manufacturer" "Yageo"
 			(at 165.1 157.48 0)
 			(effects
@@
 			)
 		)
-		(property "DigiKey" "541-49.9TCT-ND"
+		(property "DigiKey" "311-49.9LRCT-ND"
 			(at 165.1 157.48 0)
 			(effects
@@
 			)
 		)
-		(property "LCSC" "C4088942"
+		(property "LCSC" "C87044"
 			(at 165.1 157.48 0)
 			(effects
@@
 			)
 		)
-		(property "Description" "Resistor 49.9R 1% 0.5 W pulse-proof 0805"
+		(property "Description" "Resistor 49.9R 1% 0402"
 			(at 165.1 157.48 0)
 			(effects
