File: layercam/v1/ring/layercam-ring.kicad_pcb (KiCad board)
At the start: 2 copper layers, 33 x 33 mm, 11 parts, among them J1 SH 6, Q1 TEMT6000

Commit message: LayerCam v1: fixes from the power, heat and impedance checks; camera software
- 0.9 V set to 0.906 V (51k), Wi-Fi VBAT to 3.60 V (20k), IR strings 47R
- 1-22 uF capacitors X6S / X7S (105-125 C) instead of X5R (85 C), same sizes
- pair widths for 100 / 90 ohm centred in the etch tolerance; ground vias at the USB layer changes
- sim/: field-solved impedance, power budget, thermal model of the housing
- firmware/: the camera program, device tree, SDK config, slicer G-code, 108 host tests

Co-Authored-By: Claude Opus 5.5 <noreply@anthropic.com>
Claude-Session: https://claude.ai/code/session_01SRhEBojLChjJZAxgunyC3D
Parts:
- R1, R2, R3: value 39R -> 47R
Changed lines of the file:
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@@
 			)
 		)
-		(property "Value" "39R"
+		(property "Value" "47R"
 			(at 0 -1.83 130)
 			(layer "B.Fab")
@@
 			)
 		)
-		(property "LCSC" "C22198"
+		(property "LCSC" "C17969"
 			(at 0 0 130)
 			(layer "B.Fab")
@@
 			)
 		)
-		(property "Value" "39R"
+		(property "Value" "47R"
 			(at 0 -1.83 175)
 			(layer "B.Fab")
@@
 			)
 		)
-		(property "LCSC" "C22198"
+		(property "LCSC" "C17969"
 			(at 0 0 175)
 			(layer "B.Fab")
@@
 			)
 		)
-		(property "Value" "39R"
+		(property "Value" "47R"
 			(at 0 -1.83 235)
 			(layer "B.Fab")
@@
 			)
 		)
-		(property "LCSC" "C22198"
+		(property "LCSC" "C17969"
 			(at 0 0 235)
 			(layer "B.Fab")
