File: layercam/v1/ring/layercam-ring.kicad_pcb (KiCad board)
At the start: 2 copper layers, 33 x 33 mm, 11 parts, among them J1 SH 6, Q1 TEMT6000

Commit message: LayerCam v1: rebuild all three boards with their badges
The OffGrid lockup, each board's name and revision, and the US flag on
the USB-C board, on the silkscreen of every board. DRC 0/0/0 on all
three. README: the console and boot pads are no longer labelled.

Co-Authored-By: Claude Opus 5.5 <noreply@anthropic.com>
Claude-Session: https://claude.ai/code/session_01SRhEBojLChjJZAxgunyC3D
Routing:
- net LED_K: track 66.7 -> 77.9 mm, vias 3 -> 4
- net STR2_M: track 21.9 -> 25.9 mm
- net VSYS: track 76.3 -> 80.0 mm
- net ALS_VCC: track 15.5 -> 16.9 mm
- net STR1_A: track 8.82 -> 10.1 mm
- net STR3_M: track 21.4 -> 20.3 mm, vias 0 -> 2
- net STR1_M: track 21.6 -> 20.7 mm
- net ALS: track 19.7 -> 19.1 mm
