File: layercam/v1/usb/layercam-usb.kicad_pcb (KiCad board)
At the start: 2 copper layers, 22 x 16 mm, 7 parts, among them J1 USB-C, J2 SH 6, U1 USBLC6-2SC6

Commit message: LayerCam v1: fixes from the power, heat and impedance checks; camera software
- 0.9 V set to 0.906 V (51k), Wi-Fi VBAT to 3.60 V (20k), IR strings 47R
- 1-22 uF capacitors X6S / X7S (105-125 C) instead of X5R (85 C), same sizes
- pair widths for 100 / 90 ohm centred in the etch tolerance; ground vias at the USB layer changes
- sim/: field-solved impedance, power budget, thermal model of the housing
- firmware/: the camera program, device tree, SDK config, slicer G-code, 108 host tests

Co-Authored-By: Claude Opus 5.5 <noreply@anthropic.com>
Claude-Session: https://claude.ai/code/session_01SRhEBojLChjJZAxgunyC3D
Routing:
- net VSYS: track 27.0 -> 24.3 mm, vias 3 -> 2
